File: pcb_v2/pcb_v2.kicad_pcb (KiCad board)
At the start: 2 copper layers, 22 parts

Commit message: WIP second board
Parts:
- added JP1: Jumper_3_Open, Jumper:SolderJumper-3_P1.3mm_Open_Pad1.0x1.5mm, F.Cu at (113.0, 73.0)
- added JP_REV1: Jumper_3_Open, Jumper:SolderJumper-3_P1.3mm_Open_Pad1.0x1.5mm, B.Cu at (113.0, 73.0)
- added MCP_A_REV1: MCP23008-xSS, Package_SO:SSOP-20_5.3x7.2mm_P0.65mm, B.Cu at (68.0, 124.0)
- added MCP_B_REV1: MCP23008-xSS, Package_SO:SSOP-20_5.3x7.2mm_P0.65mm, B.Cu at (68.0, 89.7)
- added MCP_C_REV1: MCP23008-xSS, Package_SO:SSOP-20_5.3x7.2mm_P0.65mm, B.Cu at (113.0, 106.6)
- moved KEY_C_5 147.7 mm to (113.0, 95.5)
- moved KEY_C_4 129.0 mm to (113.0, 78.5)
- moved KEY_B_5 98.9 mm to (59.0, 78.5)
- moved MCP_B1 96.3 mm to (68.0, 89.7)
- moved KEY_C_0 95.6 mm to (113.0, 112.5)
- moved KEY_B_3 93.7 mm to (95.0, 70.0)
- moved KEY_C_2 90.0 mm to (130.5, 104.0)
- moved KEY_B_0 85.4 mm to (77.0, 95.5)
- moved KEY_B_2 84.5 mm to (95.0, 87.0)
- moved KEY_B_1 77.1 mm to (95.0, 104.0)
- moved KEY_C_3 74.0 mm to (131.0, 87.0)
- moved KEY_C_1 66.3 mm to (131.0, 121.0)
- moved MCP_A1 44.0 mm to (68.0, 124.0)
- moved MCP_C1 42.8 mm to (113.0, 106.6)
- moved KEY_A_0 36.0 mm to (77.0, 129.5)
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Connections:
- net Net-(MCP_A1-Pad3) renamed SEL
- MCP_A1 pad 9: unconnected-(MCP_A1-Pad9) -> Earth
- MCP_B1 pad 9: unconnected-(MCP_B1-Pad9) -> Earth
- MCP_C1 pad 9: unconnected-(MCP_C1-Pad9) -> Earth
Routing:
- net Earth: track 0.00 -> 600.9 mm
- net +3V3: track 0.00 -> 266.5 mm, vias 0 -> 4
- net SCL: track 0.00 -> 171.1 mm, vias 0 -> 3
- net SEL: track 0.00 -> 168.9 mm, vias 0 -> 7
- net SDA: track 0.00 -> 158.1 mm, vias 0 -> 4
- net Net-(KEY_B_3-Pad2): track 0.00 -> 47.7 mm, vias 0 -> 1
- net Net-(KEY_B_1-Pad2): track 0.00 -> 47.0 mm, vias 0 -> 1
- net Net-(KEY_C_4-Pad2): track 0.00 -> 43.8 mm, vias 0 -> 1
- net Net-(KEY_A_5-Pad2): track 0.00 -> 43.6 mm, vias 0 -> 1
- net Net-(KEY_A_2-Pad2): track 0.00 -> 43.3 mm, vias 0 -> 1
- net Net-(KEY_C_3-Pad2): track 0.00 -> 42.2 mm, vias 0 -> 1
- net Net-(KEY_C_1-Pad2): track 0.00 -> 39.5 mm, vias 0 -> 1
- net Net-(KEY_B_2-Pad2): track 0.00 -> 36.2 mm, vias 0 -> 1
- net Net-(KEY_B_4-Pad2): track 0.00 -> 33.9 mm, vias 0 -> 1
- net Net-(KEY_A_3-Pad2): track 0.00 -> 31.6 mm, vias 0 -> 1
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Other:
- board outline added: 104.5 x 75.5 mm

Commit message: WIP second board
Parts:
- moved KEY_C_2 0.50 mm to (131.0, 104.0)
Routing:
- net Net-(KEY_C_3-Pad2): track 42.2 -> 42.8 mm
Other:
- board size 104.5 x 75.5 mm -> 105 x 75.5 mm
Changed lines of the file:
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@@
     (property "Sheetname" "")
     (attr through_hole)
-    (fp_text reference "KEY_B_4" (at 0 -8.255) (layer "F.SilkS")
+    (fp_text reference "KEY_B_4" (at 0 -6.5) (layer "F.SilkS")
       (effects (font (size 1 1) (thickness 0.15)))
     )
@@
       (effects (font (size 1 1) (thickness 0.15)))
     )
-    (fp_text user "${REFERENCE}" (at 0 -8.255) (layer "B.SilkS")
+    (fp_text user "${REFERENCE}" (at 0 -6.5) (layer "B.SilkS")
       (effects (font (size 1 1) (thickness 0.15)) (justify mirror))
     )
@@
     (property "Sheetname" "")
     (attr exclude_from_pos_files)
-    (fp_text reference "JP1" (at 0 -1.8) (layer "F.SilkS")
+    (fp_text reference "JP1" (at 0 2.5) (layer "F.SilkS")
       (effects (font (size 1 1) (thickness 0.15)))
     )
@@
     (property "Sheetname" "")
     (attr through_hole)
-    (fp_text reference "KEY_C_3" (at 0 -6.5) (layer "F.SilkS")
+    (fp_text reference "KEY_C_3" (at 0 -6) (layer "F.SilkS")
       (effects (font (size 1 1) (thickness 0.15)))
     )
@@
   )
   (footprint "kailh:SW_PG1350_reversible" (layer "F.Cu")
-    (at 130.5 104)
+    (at 131 104)
     (descr "Kailh \"Choc\" PG1350 keyswitch, able to be mounted on front or back of PCB")
     (tags "kailh,choc")
@@
     (property "Sheetname" "")
     (attr through_hole)
-    (fp_text reference "KEY_A_2" (at 0 -8.255) (layer "F.SilkS")
+    (fp_text reference "KEY_A_2" (at 0 -6) (layer "F.SilkS")
       (effects (font (size 1 1) (thickness 0.15)))
     )
@@
       (effects (font (size 1 1) (thickness 0.15)))
     )
-    (fp_text user "${REFERENCE}" (at 0 -8.255) (layer "B.SilkS")
+    (fp_text user "${REFERENCE}" (at 0 -6) (layer "B.SilkS")
       (effects (font (size 1 1) (thickness 0.15)) (justify mirror))
     )
@@
     (property "Sheetname" "")
     (attr through_hole)
-    (fp_text reference "KEY_B_5" (at 0 -7) (layer "F.SilkS")
+    (fp_text reference "KEY_B_5" (at 0 -6.5) (layer "F.SilkS")
       (effects (font (size 1 1) (thickness 0.15)))
     )
@@
       (effects (font (size 1 1) (thickness 0.15)))
     )
-    (fp_text user "${REFERENCE}" (at 0 -7) (layer "B.SilkS")
+    (fp_text user "${REFERENCE}" (at 0 -6.5) (layer "B.SilkS")
       (effects (font (size 1 1) (thickness 0.15)) (justify mirror))
     )
@@
     (property "Sheetname" "")
     (attr through_hole)
-    (fp_text reference "KEY_B_3" (at 0 -7) (layer "F.SilkS")
+    (fp_text reference "KEY_B_3" (at 0 -6.5) (layer "F.SilkS")
       (effects (font (size 1 1) (thickness 0.15)))
     )
@@
       (effects (font (size 1 1) (thickness 0.15)))
     )
-    (fp_text user "${REFERENCE}" (at 0 -7) (layer "B.SilkS")
+    (fp_text user "${REFERENCE}" (at 0 -6.5) (layer "B.SilkS")
       (effects (font (size 1 1) (thickness 0.15)) (justify mirror))
     )
@@
     (property "Sheetname" "")
     (attr through_hole)
-    (fp_text reference "KEY_C_4" (at 0 -8.255) (layer "F.SilkS")
+    (fp_text reference "KEY_C_4" (at -0.5 3) (layer "F.SilkS")
       (effects (font (size 1 1) (thickness 0.15)))
     )
@@
       (effects (font (size 1 1) (thickness 0.15)))
     )
-    (fp_text user "${REFERENCE}" (at 0 -8.255) (layer "B.SilkS")
+    (fp_text user "${REFERENCE}" (at -0.5 3) (layer "B.SilkS")
       (effects (font (size 1 1) (thickness 0.15)) (justify mirror))
     )
@@
     (property "Sheetname" "")
     (attr exclude_from_pos_files)
-    (fp_text reference "JP_REV1" (at 0 1.8) (layer "B.SilkS")
+    (fp_text reference "JP_REV1" (at 0 -2.5) (layer "B.SilkS")
       (effects (font (size 1 1) (thickness 0.15)) (justify mirror))
     )
@@
   )
   (gr_arc (start 122 70) (mid 119.631372 69.605883) (end 117.5 68.5) (layer "Edge.Cuts") (width 0.1))
-  (gr_line (start 34 137) (end 84.5 137) (layer "Edge.Cuts") (width 0.1))
-  (gr_line (start 34 122) (end 34 137) (layer "Edge.Cuts") (width 0.1))
-  (gr_arc (start 86 61.5) (mid 68.558702 68.116261) (end 50 70) (layer "Edge.Cuts") (width 0.1))
+  (gr_line (start 33.5 137) (end 84.5 137) (layer "Edge.Cuts") (width 0.1))
+  (gr_line (start 33.5 122) (end 33.5 137) (layer "Edge.Cuts") (width 0.1))
+  (gr_arc (start 86 61.5) (mid 68.516196 67.936235) (end 50 70) (layer "Edge.Cuts") (width 0.1))
   (gr_arc (start 138.5 79.5) (mid 129.10765 76.734081) (end 122 70) (layer "Edge.Cuts") (width 0.1))
   (gr_line (start 123.5 128.5) (end 138.5 128.5) (layer "Edge.Cuts") (width 0.1))
@@
   (gr_line (start 86 61.5) (end 117.5 61.5) (layer "Edge.Cuts") (width 0.1))
   (gr_line (start 138.5 79.5) (end 138.5 128.5) (layer "Edge.Cuts") (width 0.1))
-  (gr_arc (start 50 70) (mid 45.784645 97.164506) (end 34 122) (layer "Edge.Cuts") (width 0.1))
+  (gr_arc (start 50 70) (mid 45.93655 97.328425) (end 33.5 122) (layer "Edge.Cuts") (width 0.1))
   (gr_line (start 117.5 61.5) (end 117.5 68.5) (layer "Edge.Cuts") (width 0.1))
   (gr_rect (start 32 121) (end 50 138) (layer "User.1") (width 0.15) (fill none))
@@
   (segment (start 113.419842 108.419842) (end 112.419842 108.419842) (width 0.25) (layer "B.Cu") (net 16))
   (segment (start 112.419842 108.419842) (end 111.6 107.6) (width 0.25) (layer "B.Cu") (net 16))
-  (segment (start 123.784991 106.948017) (end 126.5 104.233008) (width 0.25) (layer "F.Cu") (net 17))
-  (segment (start 116.490417 106.948017) (end 123.784991 106.948017) (width 0.25) (layer "F.Cu") (net 17))
-  (segment (start 126.5 91.3) (end 126 90.8) (width 0.25) (layer "F.Cu") (net 17))
+  (segment (start 126.725421 91.525421) (end 126 90.8) (width 0.25) (layer "F.Cu") (net 17))
   (segment (start 113.716265 107.487701) (end 114.255949 106.948017) (width 0.25) (layer "F.Cu") (net 17))
   (segment (start 114.255949 106.948017) (end 116.490417 106.948017) (width 0.25) (layer "F.Cu") (net 17))
-  (segment (start 126.5 104.233008) (end 126.5 91.3) (width 0.25) (layer "F.Cu") (net 17))
+  (segment (start 116.490417 106.948017) (end 124.551983 106.948017) (width 0.25) (layer "F.Cu") (net 17))
+  (segment (start 126.725421 104.774579) (end 126.725421 91.525421) (width 0.25) (layer "F.Cu") (net 17))
+  (segment (start 124.551983 106.948017) (end 126.725421 104.774579) (width 0.25) (layer "F.Cu") (net 17))
   (segment (start 126 90.8) (end 136 90.8) (width 0.25) (layer "F.Cu") (net 17))
   (segment (start 112.512299 107.487701) (end 113.716265 107.487701) (width 0.25) (layer "F.Cu") (net 17))

Commit message: WIP
Parts:
- moved JACK1 1.00 mm to (117.6, 66.5)
Routing:
- net +3V3: track 266.5 -> 269.0 mm
- net Earth: track 600.9 -> 598.5 mm
- net SDA: track 158.1 -> 160.2 mm
- net Net-(KEY_C_5-Pad2): track 22.2 -> 24.1 mm
- net Net-(KEY_B_0-Pad2): track 26.8 -> 28.4 mm
- net Net-(KEY_A_0-Pad2): track 26.7 -> 28.2 mm
- net Net-(KEY_C_1-Pad2): track 39.5 -> 40.8 mm
- net Net-(KEY_C_4-Pad2): track 43.8 -> 44.8 mm
- net SCL: track 171.1 -> 172.1 mm
- net Net-(KEY_B_5-Pad2): track 25.5 -> 26.1 mm
- net SEL: track 168.9 -> 168.4 mm
Other:
- board size 105 x 75.5 mm -> 105 x 74.5 mm
- board text added: "François Lehericey"
- board text added: "JLCJLCJLCJLC"

Commit message: WIP second board
Parts:
- removed JP_REV1: Jumper_3_Open, Jumper:SolderJumper-3_P1.3mm_Open_Pad1.0x1.5mm
- added JP_5V_BACK1: Jumper_2_Open, Jumper:SolderJumper-2_P1.3mm_Open_Pad1.0x1.5mm, B.Cu at (95.0, 81.5)
- added JP_5V_FRONT1: Jumper_2_Open, Jumper:SolderJumper-2_P1.3mm_Open_Pad1.0x1.5mm, F.Cu at (95.0, 65.5)
- added JP_GND_BACK1: Jumper_2_Open, Jumper:SolderJumper-2_P1.3mm_Open_Pad1.0x1.5mm, B.Cu at (94.8, 65.5)
- added JP_GND_FRONT1: Jumper_2_Open, Jumper:SolderJumper-2_P1.3mm_Open_Pad1.0x1.5mm, F.Cu at (95.0, 82.5)
- added JP_SELECT2: Jumper_3_Open, Jumper:SolderJumper-3_P1.3mm_Open_Pad1.0x1.5mm, B.Cu at (113.0, 73.0)
- JACK1: footprint PJ-320A:TRRS-PJ-320A-no-Fmask -> PJ-320A:TRRS-PJ-320A-no-Fmask-reversible
- turned JP_SELECT1 to 180 degrees
- renumbered JP1 to JP_SELECT1
Connections:
- JACK1 pad S: Earth -> Net-(JACK1-PadS)
- JACK1 pad T: +3V3 -> Net-(JACK1-PadT)
Routing:
- net Net-(JACK1-PadT): track 0.00 -> 41.4 mm
- net +3V3: track 269.0 -> 297.4 mm, vias 4 -> 5
- net Earth: track 598.5 -> 571.0 mm
- net Net-(JACK1-PadS): track 0.00 -> 26.6 mm
- net SDA: track 160.2 -> 159.5 mm
- net SCL: track 172.1 -> 171.5 mm
