File: pcb_v2/pcb_v2.kicad_pcb (KiCad board)
At the start: 2 copper layers, 105 x 74.5 mm, 31 parts

Commit message: pcb v2 fixes + support for v2 in firmware
Connections:
- MCP_B_REV1 pad 9: unconnected-(MCP_B_REV1-Pad9) -> Earth
- MCP_C_REV1 pad 4: Earth -> +3V3
- MCP_C_REV1 pad 9: unconnected-(MCP_C_REV1-Pad9) -> Earth
Routing:
- net Earth: track 571.0 -> 585.2 mm
- net +3V3: track 297.4 -> 303.5 mm
