File: pcb_v2/pcb_v2.kicad_sch (KiCad schematic)
At the start: 23 parts

Commit message: WIP second board
Parts:
- added JP_REV1: Jumper_3_Open, Jumper:SolderJumper-3_P1.3mm_Open_Pad1.0x1.5mm, symbol Jumper:Jumper_3_Open
- added MCP_A_REV1, MCP_B_REV1, MCP_C_REV1: MCP23008-xSS, Package_SO:SSOP-20_5.3x7.2mm_P0.65mm, symbol Interface_Expansion:MCP23008-xSS
- JACK1: value AudioJack4 -> (none); footprint PJ-320A:TRRS-PJ-320A-no-Fmask -> (none)
- JP1: value Jumper_3_Open -> (none)
Connections:
- net +3V3: now also JACK1.T, JP1.1 (A), JP_REV1.1 (A), MCP_A_REV1.20 (VDD), MCP_A_REV1.6 (~{RESET}), MCP_B_REV1.20 (VDD), MCP_B_REV1.5 (A0), MCP_B_REV1.6 (~{RESET}), MCP_C_REV1.20 (VDD), MCP_C_REV1.6 (~{RESET}); no longer JACK1.S
- net Earth: now also JACK1.S, JP1.3 (B), MCP_A1.9 (VSS), MCP_B1.9 (VSS), MCP_C1.9 (VSS), JP_REV1.3 (B), MCP_A_REV1.4 (A1), MCP_A_REV1.5 (A0), MCP_A_REV1.9 (VSS), MCP_B_REV1.4 (A1), MCP_C_REV1.4 (A1), MCP_C_REV1.5 (A0); no longer JACK1.T
- net SCL: now also MCP_A_REV1.1 (SCL), MCP_B_REV1.1 (SCL), MCP_C_REV1.1 (SCL)
- net SDA: now also MCP_A_REV1.2 (SDA), MCP_B_REV1.2 (SDA), MCP_C_REV1.2 (SDA)
- net at KEY_C_1.2 (B), MCP_C1.13 (GP1): now also MCP_C_REV1.13 (GP1)
- net at KEY_B_3.2 (B), MCP_B1.15 (GP3): now also MCP_B_REV1.15 (GP3)
- net at KEY_A_5.2 (B), MCP_A1.17 (GP5): now also MCP_A_REV1.17 (GP5)
- net at KEY_C_3.2 (B), MCP_C1.15 (GP3): now also MCP_C_REV1.15 (GP3)
- net at KEY_A_0.2 (B), MCP_A1.12 (GP0): now also MCP_A_REV1.12 (GP0)
- net at KEY_A_1.2 (B), MCP_A1.13 (GP1): now also MCP_A_REV1.13 (GP1)
- net at KEY_A_2.2 (B), MCP_A1.14 (GP2): now also MCP_A_REV1.14 (GP2)
- net at KEY_A_3.2 (B), MCP_A1.15 (GP3): now also MCP_A_REV1.15 (GP3)
- net at KEY_A_4.2 (B), MCP_A1.16 (GP4): now also MCP_A_REV1.16 (GP4)
- net SEL: now reaches JP1.2 (C), MCP_A1.3 (A2), MCP_B1.3 (A2), MCP_C1.3 (A2)
- net SEL: now also JP_REV1.2 (C), MCP_A_REV1.3 (A2), MCP_B_REV1.3 (A2), MCP_C_REV1.3 (A2)
- net at KEY_C_0.2 (B), MCP_C1.12 (GP0): now also MCP_C_REV1.12 (GP0)
- net at KEY_B_2.2 (B), MCP_B1.14 (GP2): now also MCP_B_REV1.14 (GP2)
- net at KEY_C_2.2 (B), MCP_C1.14 (GP2): now also MCP_C_REV1.14 (GP2)
- net at KEY_C_4.2 (B), MCP_C1.16 (GP4): now also MCP_C_REV1.16 (GP4)
- net at KEY_C_5.2 (B), MCP_C1.17 (GP5): now also MCP_C_REV1.17 (GP5)
- net at KEY_B_5.2 (B), MCP_B1.17 (GP5): now also MCP_B_REV1.17 (GP5)
- net at KEY_B_0.2 (B), MCP_B1.12 (GP0): now also MCP_B_REV1.12 (GP0)
- net at KEY_B_1.2 (B), MCP_B1.13 (GP1): now also MCP_B_REV1.13 (GP1)
- net at KEY_B_4.2 (B), MCP_B1.16 (GP4): now also MCP_B_REV1.16 (GP4)
Other:
- moved on the sheet: JACK1, KEY_A_0, KEY_A_1, KEY_A_2, KEY_A_3, KEY_A_4, KEY_A_5, KEY_B_0, KEY_B_1, KEY_B_2, KEY_B_3, KEY_B_4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

Commit message: WIP
Parts:
- added JP_5V_BACK, JP_GND_BACK, JP_GND_FRONT: Jumper_2_Open, symbol Jumper:Jumper_2_Open
- added JP_5V_FRONT: (no value), symbol Jumper:Jumper_2_Open
- JP1: value (none) -> Jumper_3_Open; footprint (none) -> Jumper:SolderJumper-3_P1.3mm_Open_Pad1.0x1.5mm
- JP_REV1: value Jumper_3_Open -> (none); footprint Jumper:SolderJumper-3_P1.3mm_Open_Pad1.0x1.5mm -> (none)
Connections:
- net +3V3: now also JP_5V_BACK.2 (B), JP_5V_FRONT.2 (B); no longer JACK1.T
- net Earth: now also JP_GND_BACK.2 (B), JP_GND_FRONT.2 (B); no longer JACK1.S
- new net: JACK1.T, JP_5V_BACK.1 (A), JP_GND_FRONT.1 (A)
- new net: JACK1.S, JP_5V_FRONT.1 (A), JP_GND_BACK.1 (A)

Commit message: WIP second board
Parts:
- JP_5V_BACK1: renamed from JP_5V_BACK; value Jumper_2_Open -> (none)
- JP_GND_BACK1: renamed from JP_GND_BACK; value Jumper_2_Open -> (none)
- JP_GND_FRONT1: renamed from JP_GND_FRONT; value Jumper_2_Open -> (none)
- renumbered JP_5V_FRONT to JP_5V_FRONT1, JP1 to JP_SELECT1, JP_REV1 to JP_SELECT2
Changed lines of the file:
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@@
   (symbol (lib_id "power:+3.3V") (at 64.77 111.76 0) (unit 1)
     (in_bom yes) (on_board yes) (fields_autoplaced)
-    (property "Reference" "#PWR?" (id 0) (at 64.77 115.57 0)
+    (property "Reference" "#PWR0137" (id 0) (at 64.77 115.57 0)
       (effects (font (size 1.27 1.27)) hide)
     )
@@
   (symbol (lib_id "Jumper:Jumper_3_Open") (at 90.17 33.02 0) (unit 1)
     (in_bom yes) (on_board yes) (fields_autoplaced)
-    (property "Reference" "JP1" (id 0) (at 90.17 26.67 0))
+    (property "Reference" "JP_SELECT1" (id 0) (at 90.17 26.67 0))
     (property "Value" "Jumper_3_Open" (id 1) (at 90.17 29.21 0))
     (property "Footprint" "Jumper:SolderJumper-3_P1.3mm_Open_Pad1.0x1.5mm" (id 2) (at 90.17 33.02 0)
@@
   (symbol (lib_id "power:+3.3V") (at 147.32 111.76 0) (unit 1)
     (in_bom yes) (on_board yes) (fields_autoplaced)
-    (property "Reference" "#PWR?" (id 0) (at 147.32 115.57 0)
+    (property "Reference" "#PWR0139" (id 0) (at 147.32 115.57 0)
       (effects (font (size 1.27 1.27)) hide)
     )
@@
   (symbol (lib_id "Jumper:Jumper_2_Open") (at 58.42 54.61 0) (unit 1)
     (in_bom yes) (on_board yes) (fields_autoplaced)
-    (property "Reference" "JP_GND_FRONT" (id 0) (at 58.42 48.26 0))
-    (property "Value" "Jumper_2_Open" (id 1) (at 58.42 50.8 0))
+    (property "Reference" "JP_GND_FRONT1" (id 0) (at 58.42 48.26 0))
+    (property "Value" "" (id 1) (at 58.42 50.8 0))
     (property "Footprint" "" (id 2) (at 58.42 54.61 0)
       (effects (font (size 1.27 1.27)) hide)
@@
   (symbol (lib_id "power:Earth") (at 68.58 54.61 0) (unit 1)
     (in_bom yes) (on_board yes) (fields_autoplaced)
-    (property "Reference" "#PWR?" (id 0) (at 68.58 60.96 0)
+    (property "Reference" "#PWR0135" (id 0) (at 68.58 60.96 0)
       (effects (font (size 1.27 1.27)) hide)
     )
@@
   (symbol (lib_id "Jumper:Jumper_3_Open") (at 115.57 32.385 0) (unit 1)
     (in_bom yes) (on_board yes) (fields_autoplaced)
-    (property "Reference" "JP_REV1" (id 0) (at 115.57 25.4 0))
+    (property "Reference" "JP_SELECT2" (id 0) (at 115.57 25.4 0))
     (property "Value" "" (id 1) (at 115.57 27.94 0))
     (property "Footprint" "" (id 2) (at 115.57 32.385 0)
@@
   (symbol (lib_id "Jumper:Jumper_2_Open") (at 58.42 31.75 0) (unit 1)
     (in_bom yes) (on_board yes) (fields_autoplaced)
-    (property "Reference" "JP_GND_BACK" (id 0) (at 58.42 25.4 0))
-    (property "Value" "Jumper_2_Open" (id 1) (at 58.42 27.94 0))
+    (property "Reference" "JP_GND_BACK1" (id 0) (at 58.42 25.4 0))
+    (property "Value" "" (id 1) (at 58.42 27.94 0))
     (property "Footprint" "" (id 2) (at 58.42 31.75 0)
       (effects (font (size 1.27 1.27)) hide)
@@
   (symbol (lib_id "power:+3.3V") (at 68.58 44.45 0) (unit 1)
     (in_bom yes) (on_board yes) (fields_autoplaced)
-    (property "Reference" "#PWR?" (id 0) (at 68.58 48.26 0)
+    (property "Reference" "#PWR0136" (id 0) (at 68.58 48.26 0)
       (effects (font (size 1.27 1.27)) hide)
     )
@@
   (symbol (lib_id "power:+3.3V") (at 229.87 110.49 0) (unit 1)
     (in_bom yes) (on_board yes) (fields_autoplaced)
-    (property "Reference" "#PWR?" (id 0) (at 229.87 114.3 0)
+    (property "Reference" "#PWR0138" (id 0) (at 229.87 114.3 0)
       (effects (font (size 1.27 1.27)) hide)
     )
@@
   (symbol (lib_id "Jumper:Jumper_2_Open") (at 58.42 21.59 0) (unit 1)
     (in_bom yes) (on_board yes) (fields_autoplaced)
-    (property "Reference" "JP_5V_FRONT" (id 0) (at 58.42 15.24 0))
+    (property "Reference" "JP_5V_FRONT1" (id 0) (at 58.42 15.24 0))
     (property "Value" "" (id 1) (at 58.42 17.78 0))
     (property "Footprint" "" (id 2) (at 58.42 21.59 0)
@@
   (symbol (lib_id "Jumper:Jumper_2_Open") (at 58.42 44.45 0) (unit 1)
     (in_bom yes) (on_board yes) (fields_autoplaced)
-    (property "Reference" "JP_5V_BACK" (id 0) (at 58.42 38.1 0))
-    (property "Value" "Jumper_2_Open" (id 1) (at 58.42 40.64 0))
+    (property "Reference" "JP_5V_BACK1" (id 0) (at 58.42 38.1 0))
+    (property "Value" "" (id 1) (at 58.42 40.64 0))
     (property "Footprint" "" (id 2) (at 58.42 44.45 0)
       (effects (font (size 1.27 1.27)) hide)
@@
       (reference "#PWR0134") (unit 1) (value "+3.3V") (footprint "")
     )
+    (path "/89c9524c-7e7b-4ed3-b072-0baf7e1e10bd"
+      (reference "#PWR0135") (unit 1) (value "Earth") (footprint "")
+    )
+    (path "/b9447259-ddad-453e-8cc7-4823b1562d51"
+      (reference "#PWR0136") (unit 1) (value "+3.3V") (footprint "")
+    )
     (path "/1a64cb86-658f-42ef-9648-c948f2b95042"
-      (reference "#PWR?") (unit 1) (value "+3.3V") (footprint "")
+      (reference "#PWR0137") (unit 1) (value "+3.3V") (footprint "")
+    )
+    (path "/c017fd4c-11f6-4df1-a28a-4ee8a96f0a35"
+      (reference "#PWR0138") (unit 1) (value "+3.3V") (footprint "")
     )
     (path "/75b4d7e8-1e95-48bc-9361-347f985d12e5"
-      (reference "#PWR?") (unit 1) (value "+3.3V") (footprint "")
-    )
-    (path "/89c9524c-7e7b-4ed3-b072-0baf7e1e10bd"
-      (reference "#PWR?") (unit 1) (value "Earth") (footprint "")
-    )
-    (path "/b9447259-ddad-453e-8cc7-4823b1562d51"
-      (reference "#PWR?") (unit 1) (value "+3.3V") (footprint "")
-    )
-    (path "/c017fd4c-11f6-4df1-a28a-4ee8a96f0a35"
-      (reference "#PWR?") (unit 1) (value "+3.3V") (footprint "")
+      (reference "#PWR0139") (unit 1) (value "+3.3V") (footprint "")
     )
     (path "/d1dcaffa-ed05-40d4-950f-95ceb666e2c3"
       (reference "JACK1") (unit 1) (value "AudioJack4") (footprint "PJ-320A:TRRS-PJ-320A-no-Fmask-reversible")
     )
+    (path "/f5f448b4-d707-47e8-801e-a358d23d25e8"
+      (reference "JP_5V_BACK1") (unit 1) (value "Jumper_2_Open") (footprint "Jumper:SolderJumper-2_P1.3mm_Open_Pad1.0x1.5mm")
+    )
+    (path "/c2edb813-c9b9-4b88-8859-0f202cac2525"
+      (reference "JP_5V_FRONT1") (unit 1) (value "Jumper_2_Open") (footprint "Jumper:SolderJumper-2_P1.3mm_Open_Pad1.0x1.5mm")
+    )
+    (path "/afe6e25b-a706-415c-9999-45c793ed5b5a"
+      (reference "JP_GND_BACK1") (unit 1) (value "Jumper_2_Open") (footprint "Jumper:SolderJumper-2_P1.3mm_Open_Pad1.0x1.5mm")
+    )
+    (path "/86660746-7dc6-4c10-81cb-cb27627084d7"
+      (reference "JP_GND_FRONT1") (unit 1) (value "Jumper_2_Open") (footprint "Jumper:SolderJumper-2_P1.3mm_Open_Pad1.0x1.5mm")
+    )
     (path "/54bb3b03-c9b2-493c-b048-17e2e34a337c"
-      (reference "JP1") (unit 1) (value "Jumper_3_Open") (footprint "Jumper:SolderJumper-3_P1.3mm_Open_Pad1.0x1.5mm")
-    )
-    (path "/f5f448b4-d707-47e8-801e-a358d23d25e8"
-      (reference "JP_5V_BACK") (unit 1) (value "Jumper_2_Open") (footprint "")
-    )
-    (path "/c2edb813-c9b9-4b88-8859-0f202cac2525"
-      (reference "JP_5V_FRONT") (unit 1) (value "Jumper_2_Open") (footprint "")
-    )
-    (path "/afe6e25b-a706-415c-9999-45c793ed5b5a"
-      (reference "JP_GND_BACK") (unit 1) (value "Jumper_2_Open") (footprint "")
-    )
-    (path "/86660746-7dc6-4c10-81cb-cb27627084d7"
-      (reference "JP_GND_FRONT") (unit 1) (value "Jumper_2_Open") (footprint "")
+      (reference "JP_SELECT1") (unit 1) (value "Jumper_3_Open") (footprint "Jumper:SolderJumper-3_P1.3mm_Open_Pad1.0x1.5mm")
     )
     (path "/963ef645-e9dd-4f29-9396-e96ac2e78f0c"
-      (reference "JP_REV1") (unit 1) (value "Jumper_3_Open") (footprint "Jumper:SolderJumper-3_P1.3mm_Open_Pad1.0x1.5mm")
+      (reference "JP_SELECT2") (unit 1) (value "Jumper_3_Open") (footprint "Jumper:SolderJumper-3_P1.3mm_Open_Pad1.0x1.5mm")
     )
     (path "/d931a47a-266e-421e-bb23-7213dd314c4a"
