File: pcb_host/pcb_host.kicad_pcb (KiCad board)
At the start: 2 copper layers, 44 x 53.5 mm, 5 parts, among them J1 AudioJack4, J2 AudioJack4, U1 Pico

Commit message: update pcb for host
Other:
- board text added: "JLCJLCJLCJLC"
Changed lines of the file:
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@@
   (gr_line (start 84 126.5) (end 128 126.5) (layer "Edge.Cuts") (width 0.1))
   (gr_arc (start 128 97.5) (mid 122.427832 85.80781) (end 120.5 73) (layer "Edge.Cuts") (width 0.1))
+  (gr_text "JLCJLCJLCJLC" (at 106 119.5) (layer "F.SilkS")
+    (effects (font (size 1 1) (thickness 0.15)))
+  )
   (segment (start 90 111) (end 87.225479 113.774521) (width 0.25) (layer "F.Cu") (net 1))
   (segment (start 90 103) (end 90 111) (width 0.25) (layer "F.Cu") (net 1))
